File: PCB/1222 LMNC VCO .sch (KiCad schematic (older format))
At the start: 39 parts, among them J1 POWER INPUT, J2 PCB INTERCONNECT MAIN, U1 TL074, U3 AS3340

Commit message: rescue
Parts:
- C1, C12, C2, C3, C4, C5, C6, C7: symbol Device:C -> 1222-LMNC-VCO--rescue:C-Device
- C8, C9: symbol Device:CP -> 1222-LMNC-VCO--rescue:CP-Device
- J1: symbol Connector:Conn_01x10_Male -> 1222-LMNC-VCO--rescue:Conn_01x10_Male-Connector
- J2: symbol Connector:Conn_01x12_Male -> 1222-LMNC-VCO--rescue:Conn_01x12_Male-Connector
- R1, R10, R11, R12, R13, R14, R15, R16, R17, R18, R19, R2, R22, R3, R4, R5, R6, R7, R8, R9: symbol Device:R -> 1222-LMNC-VCO--rescue:R-Device
- RV1, RV6: symbol Device:R_POT_TRIM -> 1222-LMNC-VCO--rescue:R_POT_TRIM-Device
- RV2, RV3, RV4: symbol Device:R_POT -> 1222-LMNC-VCO--rescue:R_POT-Device
- U1: symbol Amplifier_Operational:TL074 -> 1222-LMNC-VCO--rescue:TL074-Amplifier_Operational
- U3: symbol Audio:AS3340 -> 1222-LMNC-VCO--rescue:AS3340-Audio
